File: Plant-health-meter.kicad_pcb (KiCad board)
At the start: 4 copper layers, 121.2 x 25 mm, 75 parts, among them J1 Conn_01x02, J2 Conn_01x02, J3 Conn_01x04, J4 UJ2-MIBH2-4-SMT-TR, J5 Conn_01x02, Q1 AO3401A, SW1 Boot, SW2 Reset, U1 LTC4412xS6, U2 TPS62172DSG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

Commit message: More updates
Parts:
- removed the C4 at (125.9, 112.6)
- removed D1: SS14, Diode_SMD:D_SMA
- added D8: BAT54J, Diode_SMD:D_SOD-323F, F.Cu at (143.6, 115.9)
- C25: value 470p -> 1n
- D5: value SS14 -> BAT60A; footprint Diode_SMD:D_SMA -> Diode_SMD:D_SOD-323
- moved D5 14.8 mm to (130.5, 110.8), turned to 180 degrees
- moved R17 3.03 mm to (142.9, 117.4)
- moved C26 2.86 mm to (142.9, 118.4), turned to 180 degrees
- moved C5 1.95 mm to (127.8, 112.8)
- moved C2 1.90 mm to (130.9, 112.8)
- moved U2 1.70 mm to (131.9, 115.5)
- moved C6 1.66 mm to (127.3, 118.1)
- moved L2 1.65 mm to (131.1, 118.1)
- moved R4 1.52 mm to (133.4, 118.2)
- moved R15 1.24 mm to (144.2, 114.4)
- moved C1 0.65 mm to (135.2, 114.6)
- moved C23 0.35 mm to (146.2, 105.9)
- moved C24 0.35 mm to (141.0, 105.9)
- moved C25 0.35 mm to (145.2, 105.9)
- moved R14 0.35 mm to (142.4, 105.4)
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Connections:
- C26 pad 2: /MCU/CAP_TIMER -> /MCU/Soil_cap
- D5 pad 1: /MCU/CAP_TIMER -> /PWR/LOAD
- D5 pad 2: /Sensors/sensor_cap -> +5V
- R17 pad 2: /MCU/CAP_TIMER -> /MCU/Soil_cap
- TP3 pad 1: /MCU/CAP_TIMER -> /MCU/Soil_cap
- U4 pad 10: /MCU/CAP_TIMER -> /MCU/Soil_cap
Routing:
- net /MCU/Soil_cap: track 0.00 -> 38.4 mm, vias 0 -> 2
- net /MCU/CAP_TIMER: track 38.2 -> 0.00 mm, vias 2 -> 0
- net +3.3V: track 29.7 -> 34.0 mm, vias 25 -> 21
- net GND: track 37.3 -> 34.1 mm, vias 77 -> 75
- net /Sensors/Q: track 3.14 -> 1.34 mm
- net /Sensors/sensor_cap: track 8.01 -> 6.71 mm
- net Net-(U2-SW): track 1.62 -> 2.61 mm
- net /PWR/LOAD: track 0.84 -> 0.09 mm
- net Net-(U4-CHIP_EN): track 20.8 -> 21.4 mm
- added copper zone on In2.Cu, net +3.3V
- removed copper zone on B.Cu, net +3.3V
- removed copper zone on In2.Cu, net GND
Other:
- board text added: "IO6"
- board text added: "IO7"
- board text added: "Soil-cap"
- board text removed: "C-timer"
- board text removed: "MTCK"
- board text removed: "MTDO"
- board text removed: "RF"
