File: Plant-health-meter.kicad_sch (KiCad schematic)
At the start: 0 parts

Commit message: Some updates
Changed lines of the file:
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@@
 	(wire
 		(pts
-			(xy 157.48 100.33) (xy 165.1 100.33)
+			(xy 157.48 104.14) (xy 165.1 104.14)
 		)
 		(stroke
@@
 	(wire
 		(pts
-			(xy 121.92 81.28) (xy 121.92 85.09)
+			(xy 157.48 100.33) (xy 165.1 100.33)
 		)
 		(stroke
@@
 	(wire
 		(pts
-			(xy 157.48 104.14) (xy 165.1 104.14)
+			(xy 121.92 81.28) (xy 121.92 85.09)
 		)
 		(stroke
@@
 		)
 		(pin "USB_D+" bidirectional
-			(at 165.1 100.33 180)
+			(at 165.1 104.14 180)
 			(effects
 				(font
@@
 		)
 		(pin "USB_D-" bidirectional
-			(at 165.1 104.14 180)
+			(at 165.1 100.33 180)
 			(effects
 				(font

Commit message: More updates
Other:
- sheet MCU ports: added Soil_cap; removed CAP_TIMER
- sheet Sensors ports: added Soil_cap; removed CAP_TIMER
Changed lines of the file:
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@@
 			)
 		)
-		(pin "CAP_TIMER" output
+		(pin "Soil_cap" output
 			(at 129.54 74.93 270)
 			(effects
@@
 			)
 		)
-		(pin "CAP_TIMER" input
-			(at 121.92 85.09 90)
-			(effects
-				(font
-					(size 1.27 1.27)
-				)
-				(justify right)
-			)
-		)
 		(pin "USB_D-" bidirectional
 			(at 157.48 100.33 0)
@@
 			(effects
 				(font
+					(size 1.27 1.27)
+				)
+				(justify right)
+			)
+		)
+		(pin "Soil_cap" input
+			(at 121.92 85.09 90)
+			(effects
+				(font
