File: mcu.kicad_sch (KiCad schematic)
At the start: 34 parts, among them J5 Conn_01x02, SW1 Boot, SW2 Reset, U4 ESP32-C3FH4X, Y1 40MHz

Commit message: Some updates
Parts:
- removed H2: MountingHole, MountingHole:MountingHole_2.2mm_M2_DIN965_Pad, symbol Mechanical:MountingHole
- added TP3: TestPoint, TestPoint:TestPoint_Pad_D1.0mm, symbol Connector:TestPoint
Connections:
- net CAP_TIMER: now also TP3.1
Other:
- moved on the sheet: AE1, C10, C11, C12, C13, C14, C15, C16, C17, C18, C19, C20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

Commit message: More updates
Connections:
- net CAP_TIMER renamed Soil_cap
Other:
- moved on the sheet: TP3
Changed lines of the file:
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@@
 	(wire
 		(pts
+			(xy 184.15 93.98) (xy 182.88 93.98)
+		)
+		(stroke
+			(width 0)
+			(type default)
+		)
+	)
+	(wire
+		(pts
 			(xy 85.09 127) (xy 86.995 127)
 		)
@@
 	(wire
 		(pts
+			(xy 182.88 93.98) (xy 182.88 91.44)
+		)
+		(stroke
+			(width 0)
+			(type default)
+		)
+	)
+	(wire
+		(pts
 			(xy 254 115.57) (xy 254 119.38)
 		)
@@
 	(wire
 		(pts
+			(xy 184.15 95.25) (xy 184.15 93.98)
+		)
+		(stroke
+			(width 0)
+			(type default)
+		)
+	)
+	(wire
+		(pts
 			(xy 151.13 124.46) (xy 151.13 129.54)
 		)
@@
 		)
 	)
-	(hierarchical_label "CAP_TIMER"
+	(hierarchical_label "Soil_cap"
 		(shape input)
 		(at 184.15 91.44 0)
@@
 	(symbol
 		(lib_id "Connector:TestPoint")
-		(at 182.88 91.44 0)
+		(at 184.15 95.25 0)
 		(mirror x)
 		(unit 1)
@@
 		(dnp no)
 		(property "Reference" "TP3"
-			(at 182.88 97.536 90)
+			(at 184.15 101.346 90)
 			(effects
 				(font
@@
 		)
 		(property "Value" "TestPoint"
-			(at 185.42 94.742 90)
+			(at 186.69 98.552 90)
 			(effects
 				(font
@@
 		)
 		(property "Footprint" "TestPoint:TestPoint_Pad_D1.0mm"
-			(at 187.96 91.44 0)
+			(at 189.23 95.25 0)
 			(effects
 				(font
@@
 		)
 		(property "Datasheet" "~"
-			(at 187.96 91.44 0)
+			(at 189.23 95.25 0)
 			(effects
 				(font
@@
 		)
 		(property "Description" "test point"
-			(at 182.88 91.44 0)
+			(at 184.15 95.25 0)
 			(effects
 				(font
