File: pwr.kicad_sch (KiCad schematic)
At the start: 23 parts, among them J1 Conn_01x02, J2 Conn_01x02, J3 Conn_01x04, J4 USB_C_Receptacle_USB2.0, Q1 AO3401A, U1 LTC4412xS6, U2 TPS62172DSG, U3 USBLC6-2P6

Commit message: Some updates
Parts:
- removed J4: USB_C_Receptacle_USB2.0, Connector_USB:USB_C_Receptacle_HRO_TYPE-C-31-M-12, symbol Connector:USB_C_Receptacle_USB2.0
- removed R2, R3: 5.1k, Resistor_SMD:R_0402_1005Metric, symbol Device:R_Small
- added J4: UJ2-MIBH2-4-SMT-TR, UJ2-MIBH2-4-SMT-TR:CUI_UJ2-MIBH2-4-SMT-TR, symbol UJ2-MIBH2-4-SMT-TR:UJ2-MIBH2-4-SMT-TR
Connections:
- net +5V: no longer U3.5 (VBUS)
- net D+: now also U3.3 (I/O2), J4.3; no longer U3.4 (I/O2)
- net D-: now also U3.1 (I/O1), J4.2; no longer U3.6 (I/O1)
- net GND: now also J4.5, J4.SH1 (SHIELD), J4.SH2 (SHIELD), J4.SH3 (SHIELD), J4.SH4 (SHIELD), J4.SH5 (SHIELD)
- net USB_D+: now also U3.4 (I/O2); no longer U3.3 (I/O2)
- net USB_D-: now also U3.6 (I/O1); no longer U3.1 (I/O1)
- net VBUS: now reaches C3.1, L1.1
- net VBUS: now also U3.5 (VBUS), J4.1
- no-connect marks 3 -> 1
Other:
- note removed: "Remove LED from production variant"

Commit message: More updates
Parts:
- removed D1: SS14, Diode_SMD:D_SMA, symbol Diode:SS14
- added D5: BAT60A, Diode_SMD:D_SOD-323, symbol Diode:BAT60A
Connections:
- net +5V: now also D5.2 (A)
- net LOAD: now also D5.1 (K)
Other:
- note removed: "Max 28v reverse"
Changed lines of the file:
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@@
-		)
-	)
-	(text "Max 28v reverse"
-		(exclude_from_sim no)
-		(at 120.65 41.656 0)
-		(effects
-			(font
-				(size 1.27 1.27)
-			)
 		)
 	)
@@
 	)
 	(symbol
-		(lib_id "Diode:SS14")
-		(at 105.41 41.91 90)
-		(unit 1)
-		(exclude_from_sim no)
-		(in_bom yes)
-		(on_board yes)
-		(dnp no)
-		(fields_autoplaced yes)
-		(property "Reference" "D1"
-			(at 107.95 40.9574 90)
-			(effects
-				(font
-					(size 1.27 1.27)
-				)
-				(justify right)
-			)
-		)
-		(property "Value" "SS14"
-			(at 107.95 43.4974 90)
-			(effects
-				(font
-					(size 1.27 1.27)
-				)
-				(justify right)
-			)
-		)
-		(property "Footprint" "Diode_SMD:D_SMA"
-			(at 109.855 41.91 0)
-			(effects
-				(font
-					(size 1.27 1.27)
-				)
-				(hide yes)
-			)
-		)
-		(property "Datasheet" "https://www.vishay.com/docs/88746/ss12.pdf"
-			(at 105.41 41.91 0)
-			(effects
-				(font
-					(size 1.27 1.27)
-				)
-				(hide yes)
-			)
-		)
-		(property "Description" "40V 1A Schottky Diode, SMA"
-			(at 105.41 41.91 0)
-			(effects
-				(font
-					(size 1.27 1.27)
-				)
-				(hide yes)
-			)
-		)
-		(pin "2"
-		)
-		(pin "1"
-		)
-		(instances
-			(project "Plant-health-meter"
-				(path "/357055bf-c309-4d6b-a2fa-f5ee5ba59771/98819006-dc75-4aad-a220-e6960b29e68b"
-					(reference "D1")
-					(unit 1)
-				)
-			)
-		)
-	)
-	(symbol
 		(lib_id "Device:C")
 		(at 139.7 139.7 0)
@@
 					(unit 1)
 				)
+			)
+		)
+	)
+	(symbol
+		(lib_id "Diode:BAT60A")
+		(at 105.41 41.91 90)
+		(unit 1)
+		(exclude_from_sim no)
+		(in_bom yes)
+		(on_board yes)
+		(dnp no)
+		(fields_autoplaced yes)
+		(property "Reference" "D5"
+			(at 107.95 40.9574 90)
+			(effects
+				(font
+					(size 1.27 1.27)
+				)
+				(justify right)
+			)
+		)
+		(property "Value" "BAT60A"
+			(at 107.95 43.4974 90)
+			(effects
+				(font
+					(size 1.27 1.27)
+				)
+				(justify right)
+			)
+		)
+		(property "Footprint" "Diode_SMD:D_SOD-323"
+			(at 109.855 41.91 0)
+			(effects
+				(font
+					(size 1.27 1.27)
+				)
+				(hide yes)
+			)
+		)
+		(property "Datasheet" "https://www.infineon.com/dgdl/Infineon-BAT60ASERIES-DS-v01_01-en.pdf?fileId=db3a304313d846880113def70c9304a9"
+			(at 105.41 41.91 0)
+			(effects
+				(font
+					(size 1.27 1.27)
+				)
+				(hide yes)
+			)
+		)
+		(property "Description" "10V 3A High Current Recitifier Schottky Diode, SOD-323"
+			(at 105.41 41.91 0)
+			(effects
+				(font
+					(size 1.27 1.27)
+				)
+				(hide yes)
+			)
+		)
+		(pin "1"
+		)
+		(pin "2"
+		)
+		(instances
+			(project ""
+				(path "/357055bf-c309-4d6b-a2fa-f5ee5ba59771/98819006-dc75-4aad-a220-e6960b29e68b"
+					(reference "D5")
+					(unit 1)
+				)
