File: sensors.kicad_sch (KiCad schematic)
At the start: 16 parts, among them U5 BME280, U6 NE555D

Commit message: Some updates
Parts:
- removed U6: NE555D, Package_SO:SOIC-8_3.9x4.9mm_P1.27mm, symbol Timer:NE555D
- added U7: TLC555xPS, Package_SO:VSSOP-8_3x3mm_P0.65mm, symbol Timer:TLC555xPS
Connections:
- net +3.3V: now also U7.4 (R), U7.8 (VCC)
- net GND: now also U7.1 (GND)
- net Q: now also U7.3 (Q)
- net at R14.1, R16.1: now also U7.7 (DIS)
- net at C25.1, R16.2: now also U7.2 (TR), U7.6 (THR)
- net sensor_cap: now reaches D5.2 (A), R15.2, S1.1
- net at C23.1: now also U7.5 (CV)
Changed lines of the file:
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@@
+	)
+	(junction
+		(at 201.93 106.68)
+		(diameter 0)
+		(color 0 0 0 0)
 	)
 	(junction
 		(at 62.23 80.01)
-		(diameter 0)
-		(color 0 0 0 0)
-	)
-	(junction
-		(at 201.93 106.68)
 		(diameter 0)
 		(color 0 0 0 0)
@@
 		)
 	)
+	(label "sensor_cap"
+		(at 205.74 64.77 0)
+		(fields_autoplaced yes)
+		(effects
+			(font
+				(size 1.27 1.27)
+			)
+			(justify left bottom)
+		)
+	)
 	(hierarchical_label "CAP_TIMER"
 		(shape output)
@@
 	)
 	(symbol
+		(lib_id "Timer:TLC555xPS")
+		(at 189.23 101.6 0)
+		(unit 1)
+		(exclude_from_sim no)
+		(in_bom yes)
+		(on_board yes)
+		(dnp no)
+		(fields_autoplaced yes)
+		(property "Reference" "U7"
+			(at 191.4241 88.9 0)
+			(effects
+				(font
+					(size 1.27 1.27)
+				)
+				(justify left)
+			)
+		)
+		(property "Value" "TLC555xPS"
+			(at 191.4241 91.44 0)
+			(effects
+				(font
+					(size 1.27 1.27)
+				)
+				(justify left)
+			)
+		)
+		(property "Footprint" "Package_SO:VSSOP-8_3x3mm_P0.65mm"
+			(at 205.74 111.76 0)
+			(effects
+				(font
+					(size 1.27 1.27)
+				)
+				(hide yes)
+			)
+		)
+		(property "Datasheet" "http://www.ti.com/lit/ds/symlink/tlc555.pdf"
+			(at 210.82 111.76 0)
+			(effects
+				(font
+					(size 1.27 1.27)
+				)
+				(hide yes)
+			)
+		)
+		(property "Description" "Single LinCMOS Timer, 555 compatible, VSSOP-8"
+			(at 189.23 101.6 0)
+			(effects
+				(font
+					(size 1.27 1.27)
+				)
+				(hide yes)
+			)
+		)
+		(pin "4"
+		)
+		(pin "7"
+		)
+		(pin "5"
+		)
+		(pin "8"
+		)
+		(pin "6"
+		)
+		(pin "3"
+		)
+		(pin "2"
+		)
+		(pin "1"
+		)
+		(instances
+			(project ""
+				(path "/357055bf-c309-4d6b-a2fa-f5ee5ba59771/673b6cbc-4dd8-4397-ae5a-9b0518551eea"
+					(reference "U7")
+					(unit 1)
+				)
+			)
+		)
+	)
+	(symbol
 		(lib_id "Device:C")
 		(at 46.99 86.36 0)
@@
 					(unit 1)
 				)
-			)
-		)
-	)
-	(symbol
-		(lib_id "Timer:NE555D")
-		(at 189.23 101.6 0)
-		(unit 1)
-		(exclude_from_sim no)
-		(in_bom yes)
-		(on_board yes)
-		(dnp no)
-		(fields_autoplaced yes)
-		(property "Reference" "U6"
-			(at 191.4241 88.9 0)
-			(effects
-				(font
-					(size 1.27 1.27)
-				)
-				(justify left)
-			)
-		)
-		(property "Value" "NE555D"
-			(at 191.4241 91.44 0)
-			(effects
-				(font
-					(size 1.27 1.27)
-				)
-				(justify left)
-			)
-		)
-		(property "Footprint" "Package_SO:SOIC-8_3.9x4.9mm_P1.27mm"
-			(at 210.82 111.76 0)
-			(effects
-				(font
-					(size 1.27 1.27)
-				)
-				(hide yes)
-			)
-		)
-		(property "Datasheet" "http://www.ti.com/lit/ds/symlink/ne555.pdf"
-			(at 210.82 111.76 0)
-			(effects
-				(font
-					(size 1.27 1.27)
-				)
-				(hide yes)
-			)
-		)
-		(property "Description" "Precision Timers, 555 compatible, SOIC-8"
-			(at 189.23 101.6 0)
-			(effects
-				(font
-					(size 1.27 1.27)
-				)
-				(hide yes)
-			)
-		)
-		(pin "8"
-		)
-		(pin "1"
-		)
-		(pin "7"
-		)
-		(pin "2"
-		)
-		(pin "3"
-		)
-		(pin "6"
-		)
-		(pin "5"
-		)
-		(pin "4"
-		)
-		(instances
-			(project ""
-				(path "/357055bf-c309-4d6b-a2fa-f5ee5ba59771/673b6cbc-4dd8-4397-ae5a-9b0518551eea"
-					(reference "U6")
-					(unit 1)
-				)

Commit message: More updates
Parts:
- removed D5: SS14, Diode_SMD:D_SMA, symbol Diode:SS14
- added D8: BAT54J, Diode_SMD:D_SOD-323F, symbol Diode:BAT54J
- C25: value 470p -> 1n
Connections:
- net sensor_cap: now also D8.2 (A)
- net CAP_TIMER renamed Soil_cap
- net Soil_cap: now also D8.1 (K)
Other:
- moved on the sheet: C21, C22, C23, C24, C25, C26, R12, R13, R14, R15, R16, R17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
