File: PCB/LEDS.kicad_sch (KiCad schematic)
At the start: 4 parts, among them J6 Conn_02x08_Counter_Clockwise, U9 TCA9555RTWR

Commit message: Finished PCB routing and added reference designators
Parts:
- J7: renamed from J6; footprint Connector_PinHeader_1.27mm:PinHeader_2x08_P1.27mm_Vertical -> Connector_PinHeader_1.27mm:PinHeader_2x08_P1.27mm_Vertical_SMD
- renumbered C24 to C29, C23 to C30, U9 to U10
Other:
- note removed: "Check INTR signal"
- moved on the sheet: C29, C30, J7, U10

Commit message: Final touches to PCB
Parts:
- renumbered C29 to C31, C30 to C32
Changed lines of the file:
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@@
 		(dnp no)
 		(fields_autoplaced yes)
-		(property "Reference" "#PWR062"
+		(property "Reference" "#PWR063"
 			(at 135.89 143.51 0)
 			(effects
@@
 			(project ""
 				(path "/357055bf-c309-4d6b-a2fa-f5ee5ba59771/76ce39c2-8099-4ede-a2b7-8493208a9861"
-					(reference "#PWR062")
+					(reference "#PWR063")
 					(unit 1)
 				)
@@
 		(dnp no)
 		(fields_autoplaced yes)
-		(property "Reference" "#PWR060"
+		(property "Reference" "#PWR061"
 			(at 111.76 138.43 0)
 			(effects
@@
 			(project ""
 				(path "/357055bf-c309-4d6b-a2fa-f5ee5ba59771/76ce39c2-8099-4ede-a2b7-8493208a9861"
-					(reference "#PWR060")
+					(reference "#PWR061")
 					(unit 1)
 				)
@@
 		(dnp no)
 		(fields_autoplaced yes)
-		(property "Reference" "#PWR063"
+		(property "Reference" "#PWR064"
 			(at 156.21 85.09 0)
 			(effects
@@
 			(project ""
 				(path "/357055bf-c309-4d6b-a2fa-f5ee5ba59771/76ce39c2-8099-4ede-a2b7-8493208a9861"
-					(reference "#PWR063")
+					(reference "#PWR064")
 					(unit 1)
 				)
@@
 		(dnp no)
 		(fields_autoplaced yes)
-		(property "Reference" "#PWR061"
+		(property "Reference" "#PWR062"
 			(at 134.62 67.31 0)
 			(effects
@@
 			(project ""
 				(path "/357055bf-c309-4d6b-a2fa-f5ee5ba59771/76ce39c2-8099-4ede-a2b7-8493208a9861"
-					(reference "#PWR061")
+					(reference "#PWR062")
 					(unit 1)
 				)
@@
 		(dnp no)
 		(fields_autoplaced yes)
-		(property "Reference" "C30"
+		(property "Reference" "C32"
 			(at 158.75 71.12 0)
 			(effects
@@
 			(project "Plant-health-meter"
 				(path "/357055bf-c309-4d6b-a2fa-f5ee5ba59771/76ce39c2-8099-4ede-a2b7-8493208a9861"
-					(reference "C30")
+					(reference "C32")
 					(unit 1)
 				)
@@
 		(dnp no)
 		(fields_autoplaced yes)
-		(property "Reference" "C29"
+		(property "Reference" "C31"
 			(at 146.05 72.39 0)
 			(effects
@@
 			(project "Plant-health-meter"
 				(path "/357055bf-c309-4d6b-a2fa-f5ee5ba59771/76ce39c2-8099-4ede-a2b7-8493208a9861"
-					(reference "C29")
+					(reference "C31")
 					(unit 1)
 				)
@@
 		(dnp no)
 		(fields_autoplaced yes)
-		(property "Reference" "#PWR059"
+		(property "Reference" "#PWR060"
 			(at 111.76 121.92 0)
 			(effects
@@
 			(project ""
 				(path "/357055bf-c309-4d6b-a2fa-f5ee5ba59771/76ce39c2-8099-4ede-a2b7-8493208a9861"
-					(reference "#PWR059")
-					(unit 1)
-				)
+					(reference "#PWR060")
+					(unit 1)
+				)
