File: PCB/Plant-health-meter.kicad_pcb (KiCad board)
At the start: 4 copper layers, 136.2 x 25 mm, 104 parts, among them J1 Conn_01x02, J2 Conn_01x02, J3 Conn_01x02, J4 Conn_01x02, J5 USB_C_Receptacle_USB2.0_14P, J6 Conn_01x02, J7 Conn_02x08_Counter_Clockwise, Q1 AO3401A, SW1 Boot, SW2 Reset, U1 TP4057, U10 TCA9555RTWR, U2 TPS61022, U3 USBLC6-2P6, U4 LTC4412xS6, U5 TPS62172DSG, U6 ESP32-C3FH4X, U7 OPA340NA, U8 BME280, U9 ADS1115IDGS, Y1 40MHz

Commit message: Production files
Parts:
- removed the R20 at (97.2, 119.3)
- removed the R21 at (98.8, 119.3)
- removed the R3 at (146.0, 107.3)
- C10, C11: value 22p -> 15p
- C25: value 500n -> 220n; footprint Capacitor_SMD:C_0603_1608Metric -> Capacitor_SMD:C_0402_1005Metric
- L2: value 1u -> 2.2n; footprint Inductor_SMD:L_0805_2012Metric -> Inductor_SMD:L_0603_1608Metric
- R1, R2: footprint Resistor_SMD:R_0603_1608Metric -> Resistor_SMD:R_0402_1005Metric
- R14, R15, R16: value 4.7k -> 5.1k
- R19: value 500 -> 510
- R22: renamed from R24; value 500 -> 510
- moved G*** 0.57 mm to (138.2, 109.8), turned to -90 degrees
- moved C25 0.54 mm to (122.1, 116.5)
- moved D8 0.41 mm to (99.8, 117.6)
- moved L2 0.14 mm to (124.7, 108.2)
- moved R18 0.12 mm to (123.2, 116.5)
- renumbered C4 to C3, C3 to C4, D7 to D10, D8 to D3, D3 to D4, D4 to D5, D5 to D6, D9 to D7, D10 to D8, D6 to D9, R22 to R20, R23 to R21, R25 to R23, R26 to R24, R4 to R3, R27 to R4
Connections:
- C1 pad 1: /PWR/charge -> +5V
- R1 pad 2: /PWR/charge -> +5V
- U1 pad 4: /PWR/charge -> +5V
- U8 pad 5: Net-(U8-SDO) -> GND
Routing:
- net /PWR/charge: track 5.32 -> 0.00 mm
- net +5V: track 0.35 -> 5.46 mm
- net Net-(U8-SDO): track 3.33 -> 0.00 mm
- net +3.3V: track 34.2 -> 33.3 mm, vias 38 -> 37
- net +BATT: track 45.4 -> 44.4 mm
- net GND: vias 169 -> 184
- removed copper zone on F.Cu, net /PWR/charge
Other:
- board text added: "IO20"
- board text added: "Plant Health Meter v0.1"
- board text removed: "IOxx"
