File: PCB/pwr.kicad_sch (KiCad schematic)
At the start: 37 parts, among them J1 Conn_01x02, J2 Conn_01x02, J4 USB_C_Receptacle_USB2.0_14P, J7 Conn_01x02, J8 Conn_01x02, Q1 AO3401A, U1 LTC4412xS6, U2 TPS62172DSG, U3 USBLC6-2P6, U6 TPS61022, U8 TP4057

Commit message: Finished PCB routing and added reference designators
Parts:
- renumbered C29 to C1, C27 to C2, C28 to C3, C3 to C4, C4 to C5, C5 to C6, C2 to C7, C6 to C8, D6 to D1, D1 to D2, D5 to D3, D2 to D4, J7 to J1, J8 to J2, J1 to J3, J2 to J4, J4 to J5, L5 to L1, L1 to L2, L2 to L3, R18 to R1, R5 to R10, R19 to R2, R20 to R3, R22 to R4, R23 to R5, R2 to R6, R3 to R7, R1 to R8, R4 to R9, U8 to U1, U6 to U2, U1 to U4, U2 to U5

Commit message: Final touches to PCB
Parts:
- L2: footprint Inductor_SMD:L_0603_1608Metric -> Inductor_SMD:L_0805_2012Metric
Changed lines of the file:
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@@
 			)
 		)
-		(property "Footprint" "Inductor_SMD:L_0603_1608Metric"
+		(property "Footprint" "Inductor_SMD:L_0805_2012Metric"
 			(at 157.48 130.81 0)
 			(effects

Commit message: ESD protection and Boost UVLO
Parts:
- added D8: ESD9B5.0ST5G, Diode_SMD:D_SOD-923, symbol Diode:ESD9B5.0ST5G
- added R27: 10k, Resistor_SMD:R_0402_1005Metric, symbol Device:R
Connections:
- net +3.3V: now also R27.1; no longer U2.5 (EN)
- net +BATT: now also D8.2 (A2)
- net GND: now also D8.1 (A1)
- new net BOOS_EN: R27.2, U2.5 (EN)
Other:
- note added: "BOOST_EN pulled low by MCU locks battery usage. Device has to be plugged in to enable boost again."
- moved on the sheet: BT1, C1, C2, C3, C7, C8, D1, D2, D3, D4, L1, L3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

Commit message: Production files
Parts:
- removed R3: 0.3, Resistor_SMD:R_0805_2012Metric, symbol Device:R
- L2: value 1u -> 2.2n; footprint Inductor_SMD:L_0805_2012Metric -> Inductor_SMD:L_0603_1608Metric
- R1, R2: footprint Resistor_SMD:R_0603_1608Metric -> Resistor_SMD:R_0402_1005Metric
- R10: LCSC C163928 -> (none)
- renumbered C4 to C3, C3 to C4, D8 to D3, D3 to D4, D4 to D5, R4 to R3, R27 to R4
Connections:
- net charge is gone; now on net +5V: C1.1, R1.2, U1.4 (V_{CC})
Other:
- note added: "Dissipation resistor removed due to low charging current (200mA)"
Changed lines of the file:
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@@
 	(text "MODE_ = PFM"
 		(exclude_from_sim no)
-		(at 127.254 78.232 0)
+		(at 128.524 78.232 0)
 		(effects
 			(font
@@
 		)
 	)
+	(text "Dissipation resistor removed due to \nlow charging current (200mA)"
+		(exclude_from_sim no)
+		(at 79.756 33.528 0)
+		(effects
+			(font
+				(size 1.27 1.27)
+			)
+		)
+	)
 	(text "BOOST_EN pulled low by MCU locks battery usage.\nDevice has to be plugged in to enable boost again."
 		(exclude_from_sim no)
@@
 	(text "Boost output needs to be lower than usb vbus - 0.3v \n-> 4V output and Vref is 600mV\nR1 = ((Vout/Vref) - 1) * R2\nR1 = ((4v/0.6v) - 1)) * 100k = 567k = 570k standard value\n-> 4.02 V"
 		(exclude_from_sim no)
-		(at 107.95 104.902 0)
+		(at 105.156 104.902 0)
 		(effects
 			(font
@@
 	(text "3.7v Li-Ion -> 4v\nAcceptable battery voltage range:\n2.7 V to 4.35 V"
 		(exclude_from_sim no)
-		(at 107.696 96.266 0)
+		(at 105.156 96.266 0)
 		(effects
 			(font
@@
 	(wire
 		(pts
-			(xy 72.39 39.37) (xy 72.39 34.29)
-		)
-		(stroke
-			(width 0)
-			(type default)
-		)
-	)
-	(wire
-		(pts
 			(xy 129.54 80.01) (xy 129.54 81.28)
 		)
@@
 	(wire
 		(pts
-			(xy 68.58 39.37) (xy 72.39 39.37)
-		)
-		(stroke
-			(width 0)
-			(type default)
-		)
-	)
-	(wire
-		(pts
 			(xy 157.48 81.28) (xy 157.48 86.36)
 		)
@@
 	(wire
 		(pts
-			(xy 55.88 39.37) (xy 60.96 39.37)
-		)
-		(stroke
-			(width 0)
-			(type default)
-		)
-	)
-	(wire
-		(pts
 			(xy 57.15 69.85) (xy 57.15 72.39)
 		)
@@
 	(wire
 		(pts
+			(xy 59.69 39.37) (xy 55.88 39.37)
+		)
+		(stroke
+			(width 0)
+			(type default)
+		)
+	)
+	(wire
+		(pts
 			(xy 30.48 96.52) (xy 30.48 99.06)
 		)
@@
 	(wire
 		(pts
+			(xy 59.69 35.56) (xy 59.69 39.37)
+		)
+		(stroke
+			(width 0)
+			(type default)
+		)
+	)
+	(wire
+		(pts
 			(xy 67.31 168.91) (xy 67.31 171.45)
 		)
@@
 		(dnp no)
 		(fields_autoplaced yes)
-		(property "Reference" "#PWR013"
+		(property "Reference" "#PWR012"
 			(at 102.87 67.31 0)
 			(effects
@@
 			(project ""
 				(path "/357055bf-c309-4d6b-a2fa-f5ee5ba59771/98819006-dc75-4aad-a220-e6960b29e68b"
-					(reference "#PWR013")
+					(reference "#PWR012")
 					(unit 1)
 				)
@@
 		(dnp no)
 		(fields_autoplaced yes)
-		(property "Reference" "C4"
+		(property "Reference" "C3"
 			(at 154.94 135.89 0)
 			(effects
@@
 			(project "Plant-health-meter"
 				(path "/357055bf-c309-4d6b-a2fa-f5ee5ba59771/98819006-dc75-4aad-a220-e6960b29e68b"
-					(reference "C4")
+					(reference "C3")
 					(unit 1)
 				)
@@
 		(on_board yes)
 		(dnp no)
-		(property "Reference" "R27"
+		(property "Reference" "R4"
 			(at 109.2201 66.04 0)
 			(effects
@@
 			(project "Plant-health-meter"
 				(path "/357055bf-c309-4d6b-a2fa-f5ee5ba59771/98819006-dc75-4aad-a220-e6960b29e68b"
-					(reference "R27")
+					(reference "R4")
 					(unit 1)
 				)
@@
 		(lib_id "Device:Battery_Cell")
 		(at 68.58 64.77 0)
-		(mirror y)
 		(unit 1)
 		(exclude_from_sim no)
@@
 		(dnp no)
 		(property "Reference" "BT1"
-			(at 64.77 61.6584 0)
+			(at 72.39 61.6584 0)
 			(effects
 				(font
@@
 		)
 		(property "Value" "Battery_Cell"
-			(at 64.77 64.1984 0)
+			(at 72.39 64.1984 0)
 			(effects
 				(font
@@
 		(dnp no)
 		(fields_autoplaced yes)
-		(property "Reference" "#PWR012"
+		(property "Reference" "#PWR013"
 			(at 105.41 163.83 0)
 			(effects
@@
 			(project ""
 				(path "/357055bf-c309-4d6b-a2fa-f5ee5ba59771/98819006-dc75-4aad-a220-e6960b29e68b"
-					(reference "#PWR012")
+					(reference "#PWR013")
 					(unit 1)
 				)
@@
 			)
 		)
-		(property "LCSC" "C163928"
+		(property "LCSC" ""
 			(at 274.32 90.17 0)
 			(effects
@@
 		(dnp no)
 		(fields_autoplaced yes)
-		(property "Reference" "R4"
+		(property "Reference" "R3"
 			(at 102.87 144.7799 0)
 			(effects
@@
 			(project "Plant-health-meter"
 				(path "/357055bf-c309-4d6b-a2fa-f5ee5ba59771/98819006-dc75-4aad-a220-e6960b29e68b"
-					(reference "R4")
+					(reference "R3")
 					(unit 1)
 				)
@@
 	(symbol
 		(lib_id "Device:R")
-		(at 64.77 39.37 90)
-		(mirror x)
-		(unit 1)
-		(exclude_from_sim no)
-		(in_bom yes)
-		(on_board yes)
-		(dnp no)
-		(property "Reference" "R3"
-			(at 64.77 33.02 90)
-			(effects
-				(font
-					(size 1.27 1.27)
-				)
-			)
-		)
-		(property "Value" "0.3"
-			(at 64.77 35.56 90)
-			(effects
-				(font
-					(size 1.27 1.27)
-				)
-			)
-		)
-		(property "Footprint" "Resistor_SMD:R_0805_2012Metric"
-			(at 64.77 37.592 90)
-			(effects
-				(font
-					(size 1.27 1.27)
-				)
-				(hide yes)
-			)
-		)
-		(property "Datasheet" "~"
-			(at 64.77 39.37 0)
-			(effects
-				(font
-					(size 1.27 1.27)
-				)
-				(hide yes)
-			)
-		)
-		(property "Description" "Resistor"
-			(at 64.77 39.37 0)
-			(effects
-				(font
-					(size 1.27 1.27)
-				)
-				(hide yes)
-			)
-		)
-		(pin "1"
-		)
-		(pin "2"
-		)
-		(instances
-			(project "Plant-health-meter"
-				(path "/357055bf-c309-4d6b-a2fa-f5ee5ba59771/98819006-dc75-4aad-a220-e6960b29e68b"
-					(reference "R3")
-					(unit 1)
-				)
-			)
-		)
-	)
-	(symbol
-		(lib_id "Device:R")
 		(at 38.1 39.37 90)
 		(unit 1)
@@
 			)
 		)
-		(property "Footprint" "Resistor_SMD:R_0603_1608Metric"
+		(property "Footprint" "Resistor_SMD:R_0402_1005Metric"
 			(at 38.1 41.148 90)
 			(effects
@@
 		(on_board yes)
 		(dnp no)
-		(property "Reference" "D4"
+		(property "Reference" "D5"
 			(at 276.0472 76.3016 90)
 			(effects
@@
 			(project "Plant-health-meter"
 				(path "/357055bf-c309-4d6b-a2fa-f5ee5ba59771/98819006-dc75-4aad-a220-e6960b29e68b"
-					(reference "D4")
+					(reference "D5")
 					(unit 1)
 				)
@@
 		(on_board yes)
 		(dnp no)
-		(property "Reference" "D8"
+		(property "Reference" "D3"
 			(at 95.25 62.2299 90)
 			(effects
@@
 			(project ""
 				(path "/357055bf-c309-4d6b-a2fa-f5ee5ba59771/98819006-dc75-4aad-a220-e6960b29e68b"
-					(reference "D8")
+					(reference "D3")
 					(unit 1)
 				)
@@
 	(symbol
 		(lib_id "power:+5V")
-		(at 72.39 34.29 0)
+		(at 59.69 35.56 0)
 		(unit 1)
 		(exclude_from_sim no)
@@
 		(on_board yes)
 		(dnp no)
-		(property "Reference" "#PWR010"
-			(at 72.39 38.1 0)
+		(property "Reference" "#PWR09"
+			(at 59.69 39.37 0)
 			(effects
 				(font
@@
 		)
 		(property "Value" "+5V"
-			(at 70.358 29.718 0)
+			(at 57.658 30.988 0)
 			(effects
 				(font
@@
 		)
 		(property "Footprint" ""
-			(at 72.39 34.29 0)
+			(at 59.69 35.56 0)
 			(effects
 				(font
@@
 		)
 		(property "Datasheet" ""
-			(at 72.39 34.29 0)
+			(at 59.69 35.56 0)
 			(effects
 				(font
@@
 		)
 		(property "Description" ""
-			(at 72.39 34.29 0)
+			(at 59.69 35.56 0)
 			(effects
 				(font
@@
 			(project "Plant-health-meter"
 				(path "/357055bf-c309-4d6b-a2fa-f5ee5ba59771/98819006-dc75-4aad-a220-e6960b29e68b"
-					(reference "#PWR010")
+					(reference "#PWR09")
 					(unit 1)
 				)
@@
 		(dnp no)
 		(fields_autoplaced yes)
-		(property "Reference" "D3"
+		(property "Reference" "D4"
 			(at 203.2 54.9274 90)
 			(effects
@@
 			(project "Plant-health-meter"
 				(path "/357055bf-c309-4d6b-a2fa-f5ee5ba59771/98819006-dc75-4aad-a220-e6960b29e68b"
-					(reference "D3")
+					(reference "D4")
 					(unit 1)
 				)
@@
 		(dnp no)
 		(fields_autoplaced yes)
-		(property "Reference" "#PWR09"
+		(property "Reference" "#PWR010"
 			(at 71.12 179.07 0)
 			(effects
@@
 			(project "Plant-health-meter"
 				(path "/357055bf-c309-4d6b-a2fa-f5ee5ba59771/98819006-dc75-4aad-a220-e6960b29e68b"
-					(reference "#PWR09")
+					(reference "#PWR010")
 					(unit 1)
 				)
@@
 		(on_board yes)
 		(dnp no)
-		(property "Reference" "#PWR019"
+		(property "Reference" "#PWR018"
 			(at 163.83 149.86 0)
 			(effects
@@
 			(project "Plant-health-meter"
 				(path "/357055bf-c309-4d6b-a2fa-f5ee5ba59771/98819006-dc75-4aad-a220-e6960b29e68b"
-					(reference "#PWR019")
+					(reference "#PWR018")
 					(unit 1)
 				)
@@
 		(on_board yes)
 		(dnp no)
-		(property "Reference" "#PWR018"
+		(property "Reference" "#PWR019"
 			(at 168.91 111.76 0)
 			(effects
@@
 			(project "Plant-health-meter"
 				(path "/357055bf-c309-4d6b-a2fa-f5ee5ba59771/98819006-dc75-4aad-a220-e6960b29e68b"
-					(reference "#PWR018")
+					(reference "#PWR019")
 					(unit 1)
 				)
@@
 			)
 		)
-		(property "Value" "1u"
+		(property "Value" "2.2n"
 			(at 157.48 128.27 90)
 			(effects
@@
 			)
 		)
-		(property "Footprint" "Inductor_SMD:L_0805_2012Metric"
+		(property "Footprint" "Inductor_SMD:L_0603_1608Metric"
 			(at 157.48 130.81 0)
 			(effects
@@
 			)
 		)
-		(property "Footprint" "Resistor_SMD:R_0603_1608Metric"
+		(property "Footprint" "Resistor_SMD:R_0402_1005Metric"
 			(at 55.372 66.04 90)
 			(effects
@@
 		(dnp no)
 		(fields_autoplaced yes)
-		(property "Reference" "C3"
+		(property "Reference" "C4"
 			(at 161.29 76.1999 0)
 			(effects
@@
 			(project ""
 				(path "/357055bf-c309-4d6b-a2fa-f5ee5ba59771/98819006-dc75-4aad-a220-e6960b29e68b"
-					(reference "C3")
+					(reference "C4")
 					(unit 1)
 				)
